File: control_board/hardware/vasttrapi_pmu.brd (EAGLE design)
At the start: 52.4 x 29.2 mm, 20 parts, among them J2 3p-2.54, U1 TINY85-20-DIP, U2 RELAY, Y1 12MHZ

Commit message: hw rev.2
Added diode before the MCU, serial-to-usb chip and sensor
Parts:
- added D2: 1N4001, Seeed-OPL-Diode:DO-41
- moved C5 5.03 mm to (53.5, 45.8), turned to 0 degrees
Connections:
- new net V_DIODE: D2.2, J2.1, U$1.16, U1.8
- net VCC: now also D2.1; no longer J2.1, U$1.16, U1.8
Routing:
- net V_DIODE: track 0.00 -> 49.9 mm, vias 0 -> 1
- net VCC: track 75.3 -> 73.5 mm, vias 0 -> 1
Other:
- board text added: "VasttraPi Power Control Board rev.2 by Dimitris Platis"
- board text removed: "VasttraPi Power Control Board rev.1 by Dimitris Platis"
Changed lines of the file:
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@@
 <text x="53.34" y="29.2608" size="1.27" layer="22" font="vector" rot="MR0" align="bottom-center">VasttraPi
 Power Control
-Board rev.1
+Board rev.2
 by Dimitris Platis</text>
 <text x="27.432" y="39.88308125" size="1.27" layer="22" font="vector" rot="MR0" align="bottom-center">GND</text>
@@
 <element name="C2" library="Seeed-OPL-Capacitor" package="CERAMIC-2.54" value="22pf" x="48.006" y="45.8616" smashed="yes" rot="R180">
 <attribute name="MPN" value="CT4-0805CG220J101F3" x="48.006" y="45.8616" size="1.778" layer="27" rot="R180" display="off"/>
+<attribute name="NAME" x="49.022" y="46.1156" size="0.4064" layer="33" ratio="10" rot="R180"/>
 <attribute name="NAME" x="52.3494" y="46.1156" size="0.8128" layer="25" ratio="10" rot="R180"/>
-<attribute name="NAME" x="49.022" y="46.1156" size="0.4064" layer="33" ratio="10" rot="R180"/>
-<attribute name="VALUE" x="49.657" y="47.5126" size="0.4064" layer="27" ratio="10" rot="R180"/>
+<attribute name="VALUE" x="48.376840625" y="46.872521875" size="0.4064" layer="27" ratio="10" rot="R180"/>
 </element>
 <element name="C3" library="Seeed-OPL-Capacitor" package="CERAMIC-2.54" value="22pf" x="42.5196" y="45.8832" smashed="yes" rot="R180">
 <attribute name="MPN" value="CT4-0805CG220J101F3" x="42.5196" y="45.8832" size="1.778" layer="27" rot="R180" display="off"/>
+<attribute name="NAME" x="43.5356" y="46.1372" size="0.4064" layer="33" ratio="10" rot="R180"/>
 <attribute name="NAME" x="39.8526" y="46.7468" size="0.8128" layer="25" ratio="10" rot="R180"/>
-<attribute name="NAME" x="43.5356" y="46.1372" size="0.4064" layer="33" ratio="10" rot="R180"/>
-<attribute name="VALUE" x="44.1706" y="47.5342" size="0.4064" layer="27" ratio="10" rot="R180"/>
+<attribute name="VALUE" x="42.8904375" y="46.894121875" size="0.4064" layer="27" ratio="10" rot="R180"/>
 </element>
 <element name="S2" library="SparkFun-Electromechanical" package="OS" value="" x="27.0764" y="30.0228" smashed="yes">
@@
 </element>
 <element name="U$3" library="adafruit" package="OSHWLOGO_BACK_0.2" value="" x="53.34" y="38.7096"/>
-<element name="C5" library="SparkFun-Capacitors" package="CAP-PTH-SMALL-KIT" value="0.1 uF" x="58.5216" y="46.0248" smashed="yes" rot="R180">
-<attribute name="PROD_ID" value="CAP-08370" x="58.5216" y="46.0248" size="1.27" layer="27" rot="R180" display="off"/>
+<element name="C5" library="SparkFun-Capacitors" package="CAP-PTH-SMALL-KIT" value="0.1 uF" x="53.4924" y="45.826678125" smashed="yes">
+<attribute name="PROD_ID" value="CAP-08370" x="53.4924" y="45.826678125" size="1.27" layer="27" display="off"/>
+</element>
+<element name="D2" library="Seeed-OPL-Diode" package="DO-41" value="1N4001" x="62.4078" y="46.085759375" rot="R180">
+<attribute name="MPN" value="1N4001" x="62.4078" y="46.085759375" size="1.778" layer="27" rot="R180" display="off"/>
 </element>
 </elements>
@@
 <contactref element="JP3" pad="1"/>
 <contactref element="U2" pad="2"/>
-<contactref element="U$1" pad="16"/>
-<contactref element="J2" pad="1"/>
-<contactref element="U1" pad="8"/>
 <contactref element="S2" pad="2"/>
-<wire x1="35.2552" y1="35.6616" x2="33.4264" y2="33.8328" width="0.6096" layer="16"/>
 <contactref element="C4" pad="2"/>
 <wire x1="59.4714" y1="39.37" x2="59.436" y2="39.3346" width="0.6096" layer="1"/>
@@
 <wire x1="59.4714" y1="39.37" x2="47.2794" y2="39.37" width="0.6096" layer="1"/>
 <wire x1="43.571" y1="35.6616" x2="47.2794" y2="39.37" width="0.6096" layer="16"/>
-<wire x1="35.2552" y1="35.6616" x2="43.571" y2="35.6616" width="0.6096" layer="16"/>
-<wire x1="33.4264" y1="33.8328" x2="32.69488125" y2="34.56431875" width="0.6096" layer="16"/>
-<wire x1="32.69488125" y1="34.56431875" x2="28.8036" y2="34.56431875" width="0.6096" layer="16"/>
-<wire x1="24.3332" y1="35.321240625" x2="26.019759375" y2="37.0078" width="0.6096" layer="1"/>
-<wire x1="26.019759375" y1="37.0078" x2="27.8866" y2="37.0078" width="0.6096" layer="1"/>
-<wire x1="24.422559375" y1="35.321240625" x2="24.3332" y2="35.321240625" width="0.6096" layer="1"/>
-<wire x1="28.8036" y1="34.56431875" x2="27.0764" y2="32.83711875" width="0.6096" layer="16"/>
-<wire x1="27.0764" y1="32.83711875" x2="27.0764" y2="32.6674" width="0.6096" layer="16"/>
-<wire x1="27.0764" y1="32.6674" x2="26.987040625" y2="32.6674" width="0.6096" layer="1"/>
-<wire x1="26.987040625" y1="32.6674" x2="24.3332" y2="35.321240625" width="0.6096" layer="1"/>
 <wire x1="66.4182" y1="29.1928" x2="62.978721875" y2="29.1928" width="0.6096" layer="1"/>
 <wire x1="62.978721875" y1="29.1928" x2="59.527440625" y2="32.64408125" width="0.6096" layer="1"/>
 <wire x1="59.527440625" y1="32.64408125" x2="59.527440625" y2="39.313959375" width="0.6096" layer="1"/>
 <wire x1="59.527440625" y1="39.313959375" x2="59.4714" y2="39.37" width="0.6096" layer="1"/>
+<contactref element="D2" pad="1"/>
+<via x="29.123640625" y="35.524440625" extent="1-16" drill="0.6" shape="square"/>
+<wire x1="29.123640625" y1="35.524440625" x2="29.2608" y2="35.6616" width="0.6096" layer="16"/>
+<wire x1="29.2608" y1="35.6616" x2="43.571" y2="35.6616" width="0.6096" layer="16"/>
+<wire x1="71.9328" y1="42.1894" x2="68.036440625" y2="46.085759375" width="0.6096" layer="16"/>
+<wire x1="68.036440625" y1="46.085759375" x2="66.8528" y2="46.085759375" width="0.6096" layer="16"/>
+<wire x1="27.0764" y1="32.6674" x2="27.0764" y2="33.4772" width="0.6096" layer="1"/>
+<wire x1="27.0764" y1="33.4772" x2="29.123640625" y2="35.524440625" width="0.6096" layer="1"/>
 </signal>
 <signal name="VRPI">
@@
 <contactref element="C5" pad="2"/>
 <wire x1="64.5598" y1="39.0722" x2="62.0114" y2="36.5238" width="0.6096" layer="1"/>
-<wire x1="54.0968" y1="48.8012" x2="54.0968" y2="48.0112" width="0.6096" layer="1"/>
-<wire x1="56.0832" y1="46.0248" x2="57.1246" y2="46.0248" width="0.6096" layer="1"/>
-<wire x1="54.0968" y1="48.0112" x2="56.0832" y2="46.0248" width="0.6096" layer="1"/>
 <wire x1="69.7462" y1="48.888" x2="69.7462" y2="44.2586" width="0.6096" layer="1"/>
 <wire x1="69.7462" y1="44.2586" x2="68.5598" y2="43.0722" width="0.6096" layer="1"/>
-<wire x1="57.1246" y1="46.0248" x2="57.1246" y2="44.4754" width="0.6096" layer="1"/>
-<wire x1="57.1246" y1="44.4754" x2="59.436" y2="42.164" width="0.6096" layer="1"/>
-<wire x1="59.436" y1="42.164" x2="61.468" y2="42.164" width="0.6096" layer="1"/>
-<wire x1="61.468" y1="42.164" x2="64.5598" y2="39.0722" width="0.6096" layer="1"/>
+<wire x1="64.5598" y1="39.0722" x2="61.468" y2="42.164" width="0.6096" layer="1"/>
+<wire x1="58.552078125" y1="42.164" x2="54.8894" y2="45.826678125" width="0.6096" layer="1"/>
+<wire x1="61.468" y1="42.164" x2="58.552078125" y2="42.164" width="0.6096" layer="1"/>
+<wire x1="54.8894" y1="45.826678125" x2="54.8894" y2="48.0086" width="0.6096" layer="1"/>
+<wire x1="54.8894" y1="48.0086" x2="54.0968" y2="48.8012" width="0.6096" layer="1"/>
 </signal>
 <signal name="D-">
@@
 <wire x1="41.0464" y1="32.512" x2="41.0464" y2="33.8328" width="0.6096" layer="1"/>
 <wire x1="39.3192" y1="30.7848" x2="41.0464" y2="32.512" width="0.6096" layer="1"/>
-<wire x1="29.8704" y1="38.4048" x2="31.0134" y2="39.5478" width="0.6096" layer="1"/>
 <wire x1="33.2766" y1="39.5478" x2="31.0134" y2="39.5478" width="0.6096" layer="1"/>
-<wire x1="33.543240625" y1="30.7848" x2="31.04388125" y2="33.284159375" width="0.6096" layer="1"/>
-<wire x1="31.04388125" y1="35.2044" x2="29.8704" y2="36.37788125" width="0.6096" layer="1"/>
-<wire x1="29.8704" y1="36.37788125" x2="29.8704" y2="38.4048" width="0.6096" layer="1"/>
-<wire x1="31.04388125" y1="33.284159375" x2="31.04388125" y2="35.2044" width="0.6096" layer="1"/>
+<wire x1="31.04388125" y1="33.284159375" x2="33.543240625" y2="30.7848" width="0.6096" layer="1"/>
+<wire x1="29.76371875" y1="38.29811875" x2="29.76371875" y2="36.8046" width="0.6096" layer="1"/>
+<wire x1="29.76371875" y1="36.8046" x2="31.04388125" y2="35.5244375" width="0.6096" layer="1"/>
+<wire x1="31.0134" y1="39.5478" x2="29.76371875" y2="38.29811875" width="0.6096" layer="1"/>
+<wire x1="31.04388125" y1="35.5244375" x2="31.04388125" y2="33.284159375" width="0.6096" layer="1"/>
 </signal>
 <signal name="RX">
@@
 <wire x1="24.8158" y1="32.151321875" x2="24.8158" y2="32.6674" width="0.6096" layer="1"/>
 </signal>
+<signal name="V_DIODE">
+<contactref element="D2" pad="2"/>
+<contactref element="U1" pad="8"/>
+<contactref element="U$1" pad="16"/>
+<wire x1="57.9628" y1="46.085759375" x2="56.007" y2="44.129959375" width="0.6096" layer="16"/>
+<wire x1="56.007" y1="44.129959375" x2="56.007" y2="35.84448125" width="0.6096" layer="16"/>
+<wire x1="56.007" y1="35.84448125" x2="52.16651875" y2="32.004" width="0.6096" layer="16"/>
+<wire x1="52.16651875" y1="32.004" x2="38.084759375" y2="32.004" width="0.6096" layer="16"/>
+<via x="38.084759375" y="32.004" extent="1-16" drill="0.6" shape="square"/>
+<wire x1="38.084759375" y1="32.004" x2="35.2552" y2="32.004" width="0.6096" layer="1"/>
+<wire x1="35.2552" y1="32.004" x2="33.4264" y2="33.8328" width="0.6096" layer="1"/>
+<contactref element="J2" pad="1"/>
+<wire x1="33.4264" y1="33.8328" x2="29.92275" y2="33.8328" width="0.6096" layer="16"/>
+<wire x1="29.92275" y1="33.8328" x2="29.8499" y2="33.90565" width="0.6096" layer="16"/>
+<wire x1="25.748790625" y1="33.90565" x2="24.3332" y2="35.321240625" width="0.6096" layer="16"/>
+<wire x1="29.8499" y1="33.90565" x2="25.748790625" y2="33.90565" width="0.6096" layer="16"/>
+<wire x1="24.3332" y1="35.321240625" x2="26.019759375" y2="37.0078" width="0.6096" layer="1"/>
+<wire x1="26.019759375" y1="37.0078" x2="27.8866" y2="37.0078" width="0.6096" layer="1"/>
+</signal>
 </signals>
