File: control_board/hardware/vasttrapi_pmu.sch (EAGLE design)
At the start: 19 parts, among them J2 3p-2.54, U1 TINY85-20-DIP, U2 RELAY, Y1 12MHZ

Commit message: hw rev.2
Added diode before the MCU, serial-to-usb chip and sensor
Parts:
- added D2: 1N4001, Seeed-OPL-Diode:DIP-DIODE-50V-1A-1N4001(DO-41)
Connections:
- new net V_DIODE: D2.-, J2.P$1, U$1.VCC, U1.VCC
- net VCC: now also D2.+; no longer J2.P$1, U$1.VCC, U1.VCC
Changed lines of the file:
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@@
 <part name="Q1" library="SparkFun-DiscreteSemi" deviceset="TRANSISTOR_NPN" device="BC547"/>
 <part name="R1" library="SparkFun-Passives" deviceset="RESISTOR" device="PTH-1/4W" value="1KΩ"/>
-<part name="SUPPLY1" library="SparkFun-Aesthetics" deviceset="VCC" device=""/>
 <part name="GND1" library="SparkFun-Aesthetics" deviceset="GND" device=""/>
 <part name="U2" library="Itead_BP_110825.lbr" deviceset="RELAY" device=""/>
@@
 <part name="J2" library="Seeed-OPL-Connector" deviceset="DIP-BLACK-FEMALE-HEADER-VERT(3P-2.54)" device="" value="3p-2.54"/>
 <part name="GND10" library="SparkFun-Aesthetics" deviceset="GND" device=""/>
-<part name="SUPPLY5" library="SparkFun-Aesthetics" deviceset="VCC" device=""/>
-<part name="SUPPLY6" library="SparkFun-Aesthetics" deviceset="VCC" device=""/>
 <part name="D1" library="Seeed-OPL-Diode" deviceset="DIP-LED-GREEN-GREEN(2P-D5MM)" device="" value="G502DC"/>
 <part name="R2" library="SparkFun-Passives" deviceset="RESISTOR" device="PTH-1/4W" value="220Ω"/>
@@
 <part name="GND14" library="SparkFun-Aesthetics" deviceset="GND" device=""/>
 <part name="C5" library="SparkFun-Capacitors" deviceset="0.1UF-50V-20%(PTH)" device="KIT-EZ" value="0.1 uF"/>
+<part name="D2" library="Seeed-OPL-Diode" deviceset="DIP-DIODE-50V-1A-1N4001(DO-41)" device="" value="1N4001"/>
+<part name="SUPPLY9" library="SparkFun-Aesthetics" deviceset="VCC" device=""/>
 </parts>
 <sheets>
@@
 <instance part="Q1" gate="G$1" x="129.54" y="66.04" rot="R90"/>
 <instance part="R1" gate="G$1" x="129.54" y="58.42" rot="R90"/>
-<instance part="SUPPLY1" gate="G$1" x="19.05" y="102.87"/>
 <instance part="GND1" gate="1" x="119.38" y="99.06"/>
 <instance part="U2" gate="G$1" x="107.95" y="76.2" rot="R90"/>
@@
 <instance part="J2" gate="G$1" x="13.97" y="34.29" rot="R270"/>
 <instance part="GND10" gate="1" x="7.62" y="48.26" rot="R270"/>
-<instance part="SUPPLY5" gate="G$1" x="17.78" y="48.26" rot="R270"/>
-<instance part="SUPPLY6" gate="G$1" x="17.78" y="66.04" rot="R180"/>
 <instance part="D1" gate="G$1" x="99.06" y="100.33" rot="R180"/>
 <instance part="R2" gate="G$1" x="90.17" y="100.33" rot="R180"/>
@@
 <instance part="GND14" gate="1" x="109.22" y="123.19" rot="R90"/>
 <instance part="C5" gate="G$1" x="106.68" y="114.3"/>
+<instance part="D2" gate="G$1" x="15.24" y="127" rot="R270"/>
+<instance part="SUPPLY9" gate="G$1" x="15.24" y="132.08"/>
 </instances>
 <busses>
@@
 </segment>
 <segment>
-<pinref part="U$1" gate="G$1" pin="VCC"/>
-<pinref part="SUPPLY1" gate="G$1" pin="VCC"/>
-<wire x1="19.05" y1="102.87" x2="19.05" y2="99.06" width="0.1524" layer="91"/>
-</segment>
-<segment>
-<pinref part="J2" gate="G$1" pin="P$1"/>
-<pinref part="SUPPLY5" gate="G$1" pin="VCC"/>
-<wire x1="17.78" y1="48.26" x2="17.78" y2="41.91" width="0.1524" layer="91"/>
-</segment>
-<segment>
-<pinref part="U1" gate="G$1" pin="VCC"/>
-<pinref part="SUPPLY6" gate="G$1" pin="VCC"/>
-<wire x1="17.78" y1="66.04" x2="25.4" y2="66.04" width="0.1524" layer="91"/>
-</segment>
-<segment>
 <pinref part="S2" gate="G$1" pin="2"/>
 <pinref part="SUPPLY7" gate="G$1" pin="VCC"/>
@@
 <pinref part="U2" gate="G$1" pin="ON"/>
 <pinref part="SUPPLY4" gate="G$1" pin="VCC"/>
+</segment>
+<segment>
+<pinref part="SUPPLY9" gate="G$1" pin="VCC"/>
+<pinref part="D2" gate="G$1" pin="+"/>
+<wire x1="15.24" y1="130.81" x2="15.24" y2="132.08" width="0.1524" layer="91"/>
 </segment>
 </net>
@@
 </segment>
 </net>
+<net name="V_DIODE" class="0">
+<segment>
+<pinref part="D2" gate="G$1" pin="-"/>
+<wire x1="15.24" y1="123.19" x2="15.24" y2="119.38" width="0.1524" layer="91"/>
+<label x="15.24" y="119.38" size="1.778" layer="95"/>
+</segment>
+<segment>
+<pinref part="U1" gate="G$1" pin="VCC"/>
+<wire x1="17.78" y1="66.04" x2="25.4" y2="66.04" width="0.1524" layer="91"/>
+<label x="13.97" y="67.31" size="1.778" layer="95"/>
+</segment>
+<segment>
+<pinref part="U$1" gate="G$1" pin="VCC"/>
+<wire x1="19.05" y1="102.87" x2="19.05" y2="99.06" width="0.1524" layer="91"/>
+<label x="19.05" y="104.14" size="1.778" layer="95"/>
+</segment>
+<segment>
+<pinref part="J2" gate="G$1" pin="P$1"/>
+<wire x1="17.78" y1="48.26" x2="17.78" y2="41.91" width="0.1524" layer="91"/>
+<label x="17.78" y="44.45" size="1.778" layer="95"/>
+</segment>
+</net>
